File: unnamed-3k-v2.kicad_pcb (KiCad board)
At the start: 2 copper layers, 59.3 x 63 mm, 31 parts, among them SW1 SW_Push, U1 ATmega32U2-AU, U2 PRTR5V0U2X, Y1 Crystal_GND24_Small

Commit message: everything else
Parts:
- moved C6 29.9 mm to (101.6, 76.1), turned to 180 degrees
- moved C4 18.8 mm to (91.6, 119.2), turned to 225 degrees
- moved C7 13.6 mm to (87.2, 81.5)
- moved C8 13.6 mm to (68.2, 81.5)
- moved C9 13.0 mm to (106.9, 81.5)
- moved F1 2.76 mm to (101.3, 72.6)
- moved C5 2.47 mm to (103.7, 106.5)
- moved C1 2.45 mm to (97.4, 100.2)
- moved R2 1.50 mm to (100.1, 102.2)
- moved R1 1.49 mm to (101.6, 103.7)
- moved C2 1.48 mm to (105.4, 111.2), turned to 135 degrees
- moved U2 1.40 mm to (93.1, 72.0)
- moved R3 1.35 mm to (79.1, 109.5), turned to 270 degrees
- moved SW1 1.35 mm to (73.2, 110.3)
- moved R4 1.32 mm to (87.5, 115.7)
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Routing:
- net GND: track 353.7 -> 161.7 mm, vias 5 -> 10
- net +5V: track 220.7 -> 190.9 mm, vias 2 -> 3
- net COL2: track 46.9 -> 57.5 mm
- net COL1: track 28.2 -> 36.0 mm, vias 2 -> 0
- net XTAL1: track 9.32 -> 13.6 mm
- net D+: track 50.5 -> 46.3 mm
- net D-: track 50.1 -> 46.1 mm
- net SWITCHLED: track 34.1 -> 30.3 mm, vias 2 -> 0
- net Net-(C1-Pad1): track 3.57 -> 5.49 mm
- net VCC: track 24.4 -> 26.3 mm
- net Net-(D2-Pad1): track 32.4 -> 30.6 mm
- net Net-(R4-Pad2): track 2.63 -> 4.43 mm
- net Net-(R3-Pad2): track 22.5 -> 20.9 mm
- net XTAL2: track 7.08 -> 8.32 mm
- net UNDERGLOWLED: track 13.1 -> 12.2 mm
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